File: usbToGB_Adapter.kicad_sch (KiCad schematic)
At the start: 17 parts, among them J2 1054500101, U1 LAN7800/Y9X, U2 HD3SS3220RNHR, U3 AP2112K-3.3, U4 AP2127K-2.5

Commit message: feat
add complete schematic and initial 4-layer PCB layout
Parts:
- removed C14, C15, C16, C17, C18, C19, C20, C21: 100nF, symbol Device:C
- removed J2: 1054500101, 1054500101:MOLEX_1054500101, symbol 1054500101:1054500101
- removed R3, R5: 900K, symbol Device:R
- removed R4: 200K, symbol Device:R
- removed U1: LAN7800/Y9X, lan7800:SQFN48_7X7_Y9X_MCH, symbol lan7800:LAN7800_Y9X
- removed U2: HD3SS3220RNHR, RNH0030A, symbol HD3SS3220RNHR:HD3SS3220RNHR
- removed U4: AP2127K-2.5, Package_TO_SOT_SMD:SOT-23-5, symbol Regulator_Linear:AP2127K-2.5
- added C1, C2: 4.7uF, Capacitor_SMD:C_0805_2012Metric, symbol Device:C
- added C10, C11, C12, C22, C23, C24, C25, C28, C29, C3, C30, C31, C32, C33, C34, C35, C36, C37, C40, C42, C8, C9: 100nF, Capacitor_SMD:C_0603_1608Metric, symbol Device:C
- added C26, C27: 12pF, Capacitor_SMD:C_0603_1608Metric, symbol Device:C
- added C38, C39, C47: 1uF, Capacitor_SMD:C_0603_1608Metric, symbol Device:C
- added C4, C43, C6: 10uF, Capacitor_SMD:C_0805_2012Metric, symbol Device:C
- added C41: 22uF, Capacitor_SMD:C_0805_2012Metric, symbol Device:C
- added C44, C5, C7: 100nF, Capacitor_SMD:C_0805_2012Metric, symbol Device:C
- added C45, C46: 100nF, Capacitor_SMD:C_0402_1005Metric, symbol Device:C
- added C48: 10nF, Capacitor_SMD:C_0603_1608Metric, symbol Device:C
- added C49, C52: TBE, Capacitor_SMD:C_1210_3225Metric, symbol Device:C
- added C50, C51, C53, C54: TBE, Capacitor_SMD:C_1206_3216Metric, symbol Device:C
- added CR1, CR2, CR3: 824012823, 824012823:DFN_012823_WRE, symbol 2026-07-16_19-35-54:824012823
- added D1: 20V, Capacitor_SMD:C_0805_2012Metric, symbol Device:D_TVS
- added D2: LED, LED_SMD:LED_0603_1608Metric, symbol Device:LED
- added FB1, FB2: 110R@100MHz, Inductor_SMD:L_1206_3216Metric, symbol Device:FerriteBead
- added FB3: 110R@100MHz, Inductor_SMD:L_0603_1608Metric, symbol Device:FerriteBead
- added J5: 1054500101, usb-c_2:MOLEX_1054500101, symbol 1054500101:1054500101
- added L1: 1.2uH, 74438336012:IND_WE-MAPI_3020_WRE, symbol Device:L
- added L2, L3: L_Coupled, 7442335600:CHIP_35600_WRE, symbol Device:L_Coupled
- added L4: L_Coupled, 744232090:SMT_32090_WRE, symbol Device:L_Coupled
- added L5: 3.3uH, 74404032033:IND_WE-LQS_3015_WRE, symbol Device:L
- added R1, R6: 330R, Resistor_SMD:R_0603_1608Metric, symbol Device:R
- added R10, R11, R17, R18: 10K, Resistor_SMD:R_0603_1608Metric, symbol Device:R
- added R12, R13, R14, R15: 2K, Resistor_SMD:R_0603_1608Metric, symbol Device:R
- added R2: 10k, Resistor_SMD:R_0603_1608Metric, symbol Device:R
- added R7: 12k, Resistor_SMD:R_0603_1608Metric, symbol Device:R
- added R9: 5k1, Resistor_SMD:R_0603_1608Metric, symbol Device:R
- added T1: WE-RJ45_7499111121A, rj45(a):7499111121A, symbol WE-RJ45_7499111121A:WE-RJ45_7499111121A
- added TP1, TP2: TestPoint, TestPoint:TestPoint_Pad_D2.0mm, symbol Connector:TestPoint
- added U1: 93AA66C-I/SN, eeprom:SOIC8-N_MC_MCH, symbol 93AA66C-L/SN:93AA66C-I_SN
- added U5: LAN7800/Y9X, lan7800:SQFN48_7X7_Y9X_MCH, symbol lan7800:LAN7800_Y9X
- added Y1: 25MHz, Crystal:Crystal_SMD_3225-4Pin_3.2x2.5mm_HandSoldering, symbol Device:Crystal
- C13: footprint (none) -> Capacitor_SMD:C_0603_1608Metric
Connections:
- net tx1+ is gone; now on net 3v3_board: C13.1
- net GND: now also C13.2, U3.2 (GND), C1.1, C10.2, C11.2, C12.2, C2.1, C22.2, C23.2, C24.2, C25.2, C26.2, C27.2, C28.2, C29.2, C3.1, C30.2, C31.2, C32.2, C33.2, C34.2, C35.2, C36.2, C37.2, C38.2, C39.2, C4.2, C40.2, C41.2, C42.2, C43.2, C47.2, C49.1, C5.2, C50.1, C51.1, C52.1, C53.1, C54.1, C6.2, C7.2, C8.2, C9.2, CR1.3 (GND), CR2.3 (GND), CR3.3 (GND), D1.1 (A1), D2.1 (K), J5.A1 (GND), J5.A12 (GND), J5.B1 (GND), J5.B12 (GND), R1.1, R12.2, R17.2, R18.2, R7.2, R9.2, U1.5 (VSS), U5.34 (TEST), U5.49 (VSS)
- net 5v_Board: now reaches U3.1 (VIN)
- net 5v_Board: now also C4.1, D1.2 (A2), FB2.2, R2.1
- net at U3.3 (EN): now also C5.1, R2.2
- net 3v3_board: now reaches U3.5 (VOUT)
- net 3v3_board: now also C23.1, C24.1, C25.1, C28.1, C29.1, C30.1, C31.1, C32.1, C33.1, C34.1, C35.1, C36.1, C39.1, C40.1, C41.1, C42.1, C43.1, C48.1, C6.1, C7.1, FB3.1, L5.2, R10.1, R11.1, R13.2, R14.2, R15.2, R6.1, U1.8 (VCC), U5.14 (VDD_SW_IN), U5.15 (VDD12_SW_FB), U5.20 (VDDVARIO), U5.21 (VDD12CORE), U5.30 (VDD12A), U5.36 (VDDVARIO), U5.38 (VDD33A), U5.39 (VDDVARIO), U5.42 (VDD12CORE), U5.44 (VDD12A), U5.46 (VDD33_REG_IN)
- new net: C45.2, L2.2
- new net: C46.2, L2.4
- new net: R11.2, U5.35 (RESET_N/PME_CLEAR)
- new net: C26.1, U5.41 (XO), Y1.1
- new net: C27.1, U5.40 (XI), Y1.2
- new net: L5.1, U5.13 (SW_OUT)
- new net: T1.1 (D1+), U5.1 (TR0P)
- new net: R14.1, T1.11
- new net: R15.1, T1.13
- new net: T1.2 (D1-), U5.2 (TR0N)
- new net: T1.3 (D2+), U5.4 (TR1P)
- new net: T1.4 (D3+), U5.7 (TR2P)
- new net: T1.5 (D3-), U5.8 (TR2N)
- new net: T1.6 (D2-), U5.5 (TR1N)
- new net: T1.7 (D4+), U5.10 (TR3P)
- new net: T1.8 (D4-), U5.11 (TR3N)
- new net: R17.1, U1.6 (ORG)
- new net: D2.2 (A), R6.2
- new net: R12.1, U5.47 (REF_REXT)
- new net: C1.2, FB1.2, L1.1
- new net: R7.1, U5.37 (USBRBIAS)
- new net: R13.1, U5.22 (PME_N/GPIO4)
- new net: TP1.1, U5.43 (PME_MODE/GPIO7)
- new net: J5.A5 (CC1), R9.1
- new net: C37.1, FB3.2, U5.25 (VDD12A)
- new net: C2.2, FB2.1, L1.2
- new net: C47.1, U5.48 (REF_FILT)
- new net: R10.2, U5.23 (VBUS_DET)
- new net CLK: U1.2 (CLK), U5.19 (EECLK/LED1/GPIO3)
- new net CS: R18.1, U1.1 (CS), U5.16 (EECS/GPIO0)
- new net D0: U1.4 (DO), U5.17 (EEDI/GPIO1)
- new net D1: U1.3 (DI), U5.18 (EEDO/LED0/GPIO2)
- new net Earth: C3.2, C44.1, C48.2, C49.2, C50.2, C51.2, C52.2, C53.2, C54.2, J5.SH1 (SHIELD3), J5.SH2 (SHIELD4), J5.SH3 (SHIELD1), J5.SH4 (SHIELD2), R1.2, T1.S1 (SHIELD1), T1.S2 (SHIELD2)
- new net LED2: T1.12, U5.24 (SUSPEND_N/LED2/GPIO5)
- new net LED3: T1.14, U5.33 (LED3/GPIO6)
- new net PHY_AVDD: T1.9 (VCC), TP2.1
- new net USB2D1_N: CR3.2 (I/O_2), J5.A7 (D-), J5.B7 (D-), L4.3
- new net USB2D1_P: CR3.1, J5.A6 (D+), J5.B6 (D+), L4.1
- new net USB2D_N: L4.2, U5.27 (USB2_DM)
- new net USB2D_P: L4.4, U5.26 (USB2_DP)
- new net USB3RX1_N: CR2.1, J5.B10 (RX1-), L3.3
- new net USB3RX1_P: CR2.2 (I/O_2), J5.B11 (RX1+), L3.1
- new net USB3RX_N: L3.4, U5.32 (USB3_RXDM)
- new net USB3RX_P: L3.2, U5.31 (USB3_RXDP)
- new net USB3TX1_N: CR1.2 (I/O_2), J5.A3 (TX1-), L2.3
- new net USB3TX1_P: CR1.1, J5.A2 (TX1+), L2.1
- new net USB3TX_N: C46.1, U5.29 (USB3_TXDM)
- new net USB3TX_P: C45.1, U5.28 (USB3_TXDP)
- new net VBUS: C44.2, FB1.1, J5.A4 (VBUS), J5.A9 (VBUS), J5.B4 (VBUS), J5.B9 (VBUS)
- new net VDD25: C10.1, C11.1, C12.1, C22.1, C38.1, C8.1, C9.1, U5.12 (VDD25A), U5.3 (VDD25A), U5.45 (VDD25_REG_OUT), U5.6 (VDD25A), U5.9 (VDD25A)
- no-connect marks 3 -> 17
Other:
- title: (none) -> GB_ethernet_to_usbC
- moved on the sheet: U3
